Commit message: arm urdf is a little wierd, but should be fine to dive into moveit setup

File: src/arm1/urdf/arm1.urdf (robot description, URDF)
Before this commit: robot arm1, 7 links, 6 joints
Links:
- added link base_base_link
Joints:
- added joint base_joint: type fixed, parent base_base_link, child base_link, origin xyz=0.75729581407264 0.598615888399153 0.307790852884674 rpy=0 0 0
- joint joint_turntable: origin xyz=-0.0 -0.0 -0.0 rpy=0 0 -1.5707963267949 -> xyz=-0.75729581407264 -0.598615888399153 -0.307790852884674 rpy=0 0 -1.5707963267949

Commit message: finally, got new arm urdf working with inverse kin. now ready to transition to real hardware, will tune in firmware for ik. ideally we will only control arm via moveit, regardless of ik or fk source ws_moveit/, not ws_moveit2

File: src/arm1/urdf/arm1.urdf (robot description, URDF)
Before this commit: robot arm1, 8 links, 7 joints
Joints:
- joint joint_turntable: limit (none) -> lower=-1.4 upper=1.4 effort=5.0 velocity=2.0; type continuous -> revolute

Commit message: made offset for joints added limits in for urdf

File: src/arm1/urdf/arm1.urdf (robot description, URDF)
Before this commit: robot arm1, 8 links, 7 joints
Joints:
- joint joint_axis1: limit (none) -> lower=-1.091 upper=1.409 effort=5.0 velocity=2.0; type continuous -> revolute
- joint joint_axis2: limit (none) -> lower=-0.696 upper=1.74746 effort=5.0 velocity=2.0; type continuous -> revolute
- joint joint_axis3: limit (none) -> lower=-1.59659 upper=1.545 effort=5.0 velocity=2.0; type continuous -> revolute
- joint joint_axis4: limit (none) -> lower=-1.002 upper=2.03959265359 effort=5.0 velocity=2.0; type continuous -> revolute
- joint joint_ender: type continuous -> revolute
- joint joint_turntable: limit lower=-1.4 upper=1.4 effort=5.0 velocity=2.0 -> lower=-1.308 upper=1.83359 effort=5.0 velocity=2.0

Commit message: virtual arm tuned to limits of actual arm with offset in armSerialInterface

File: src/arm1/urdf/arm1.urdf (robot description, URDF)
Before this commit: robot arm1, 8 links, 7 joints
Joints:
- joint joint_axis3: limit lower=-1.59659 upper=1.545 effort=5.0 velocity=2.0 -> lower=-1.33479 upper=1.8067995 effort=5.0 velocity=2.0
- joint joint_ender: limit (none) -> lower=-1.375 upper=0.76459265359 effort=5.0 velocity=2.0
- joint joint_turntable: limit lower=-1.308 upper=1.83359 effort=5.0 velocity=2.0 -> lower=-2.03859 upper=0.984 effort=5.0 velocity=2.0
