Commit message: weewaa

File: src/arm2_moveit_config/config/arm2.ros2_control.xacro (robot description, xacro)
@@ -1,5 +1,5 @@
 <?xml version="1.0"?>
 <robot xmlns:xacro="http://www.ros.org/wiki/xacro">
-    <xacro:macro name="arm1_ros2_control" params="name initial_positions_file">
+    <xacro:macro name="arm2_ros2_control" params="name initial_positions_file">
         <xacro:property name="initial_positions" value="${load_yaml(initial_positions_file)['initial_positions']}"/>
         <ros2_control name="${name}" type="system">

File: src/arm2_moveit_config/config/arm2.urdf.xacro (robot description, xacro)
@@ -1,9 +1,9 @@
 <?xml version="1.0"?>
-<robot xmlns:xacro="http://www.ros.org/wiki/xacro" name="arm1">
+<robot xmlns:xacro="http://www.ros.org/wiki/xacro" name="arm2">
     <xacro:arg name="initial_positions_file" default="initial_positions.yaml" />
     <!-- Import arm1 urdf file -->
     <xacro:include filename="$(find arm1)/urdf/arm1.urdf" />
     <!-- Import control_xacro -->
-    <xacro:include filename="arm1.ros2_control.xacro" />
-    <xacro:arm1_ros2_control name="FakeSystem" initial_positions_file="$(arg initial_positions_file)"/>
+    <xacro:include filename="arm2.ros2_control.xacro" />
+    <xacro:arm2_ros2_control name="FakeSystem" initial_positions_file="$(arg initial_positions_file)"/>
 </robot>
