Commit message: urdf is messed up, but we have a proper display launcher now

File: src/rover_urdfs/urdf/Full_Assembly.urdf (robot description, URDF)
Before this commit: robot Full_Assembly, 11 links, 10 joints
Links:
- removed link Arm
- removed link Back_Bogie
- removed link Back_Bogie_Left_Wheel
- removed link Back_Bogie_Right_Wheel
- removed link Chassis_Frame
- removed link Left_Bogie
- removed link Left_Bogie_Back_Wheel
- removed link Left_Bogie_Front_Wheel
- removed link Right_Bogie
- removed link Right_Bogie_Back_Wheel
- removed link Right_Bogie_Front_Wheel
- added link arm_link, mass 0.232083853065316; collision mesh filename=package://rover_urdfs/meshes/Arm.STL; visual mesh filename=package://rover_urdfs/meshes/Arm.STL
- added link back_bogie, mass 2.03126342918492; collision mesh filename=package://rover_urdfs/meshes/Back_Bogie.STL; visual mesh filename=package://rover_urdfs/meshes/Back_Bogie.STL
- added link back_bogie_left_wheel, mass 4.54890356187038; collision mesh filename=package://rover_urdfs/meshes/Back_Bogie_Left_Wheel.STL; visual mesh filename=package://rover_urdfs/meshes/Back_Bogie_Left_Wheel.STL
- added link back_bogie_right_wheel, mass 4.54890356187038; collision mesh filename=package://rover_urdfs/meshes/Back_Bogie_Right_Wheel.STL; visual mesh filename=package://rover_urdfs/meshes/Back_Bogie_Right_Wheel.STL
- added link base_link
- added link chassis_frame, mass 16.2612895685876; collision mesh filename=package://rover_urdfs/meshes/Chassis_Frame.STL; visual mesh filename=package://rover_urdfs/meshes/Chassis_Frame.STL
- added link left_bogie, mass 3.34124121849343; collision mesh filename=package://rover_urdfs/meshes/Left_Bogie.STL; visual mesh filename=package://rover_urdfs/meshes/Left_Bogie.STL
- added link left_bogie_back_wheel, mass 4.54890356187038; collision mesh filename=package://rover_urdfs/meshes/Left_Bogie_Back_Wheel.STL; visual mesh filename=package://rover_urdfs/meshes/Left_Bogie_Back_Wheel.STL
- added link left_bogie_front_wheel, mass 4.54890356187038; collision mesh filename=package://rover_urdfs/meshes/Left_Bogie_Front_Wheel.STL; visual mesh filename=package://rover_urdfs/meshes/Left_Bogie_Front_Wheel.STL
- added link right_bogie, mass 3.34124121849343; collision mesh filename=package://rover_urdfs/meshes/Right_Bogie.STL; visual mesh filename=package://rover_urdfs/meshes/Right_Bogie.STL
- added link right_bogie_back_wheel, mass 4.54890356187038; collision mesh filename=package://rover_urdfs/meshes/Right_Bogie_Back_Wheel.STL; visual mesh filename=package://rover_urdfs/meshes/Right_Bogie_Back_Wheel.STL
- added link right_bogie_front_wheel, mass 4.54890356187038; collision mesh filename=package://rover_urdfs/meshes/Right_Bogie_Front_Wheel.STL; visual mesh filename=package://rover_urdfs/meshes/Right_Bogie_Front_Wheel.STL
Joints:
- removed joint Arm
- removed joint Back_Connect
- removed joint Back_Connect_Left
- removed joint Back_Connect_Right
- removed joint Left_Connect
- removed joint Left_Connect_Back
- removed joint Left_Connect_Front
- removed joint Right_Connect
- removed joint Right_Connect_Back
- removed joint Right_Connect_Front
- added joint arm_joint: type fixed, parent chassis_frame, child arm_link, origin xyz=0.0726472931247326 0.0460194024352475 -0.0975250000000328 rpy=3.14159265358979 0 2.20588191770284, axis 0 0 0
- added joint back_connect: type continuous, parent chassis_frame, child back_bogie, origin xyz=0.055470277282733 -0.512439057564754 -0.421614058115213 rpy=1.5602438137183 -0.0105513381921141 -1.57068498159409, axis -0.999772994789274 0.0211020967603054 0
- added joint back_connect_left: type continuous, parent back_bogie, child back_bogie_left_wheel, origin xyz=0 -0.000691989544948202 0.327180673083095 rpy=3.14159265358979 0 3.12048880228838, axis 0.00011133900256751 0.0105511424118299 0.999944328949083
- added joint back_connect_right: type continuous, parent back_bogie, child back_bogie_right_wheel, origin xyz=-3.02068909376896E-05 -0.0028625836475128 -0.356845710106984 rpy=3.14159265358926 0 -0.0105519256507057, axis 0 0.0105517298382485 -0.999944328949077
- added joint base_joint: type fixed, parent base_link, child chassis_frame, origin xyz=0.0726472931247326 0.0460194024352475 -0.0975250000000328 rpy=0 0 0
- added joint left_connect: type continuous, parent chassis_frame, child left_bogie, origin xyz=-0.248729166875268 0.369784478188223 -0.345807860434498 rpy=0.51304684994759 0 3.14159265358979, axis 0 0 1
- added joint left_connect_back: type continuous, parent left_bogie, child left_bogie_back_wheel, origin xyz=0.0829250000000004 0.32306401672449 -0.274881622694233 rpy=-1.5707963267949 0.51304684994759 1.5707963267949, axis 1 0 0
- added joint left_connect_front: type continuous, parent left_bogie, child left_bogie_front_wheel, origin xyz=0.0829250000000001 -0.0743919967284671 -0.0455554713072941 rpy=1.5707963267949 0.618626537467851 1.5707963267949, axis 0.994431640250643 0.105383646114637 0
- added joint right_connect: type continuous, parent chassis_frame, child right_bogie, origin xyz=0.365966373124733 0.366267486623604 -0.182466340171182 rpy=1.5707963267949 0 1.5707963267949, axis 0 0 1
- added joint right_connect_back: type continuous, parent right_bogie, child right_bogie_back_wheel, origin xyz=-0.406064141803662 -0.239545992505552 0.11109638 rpy=0 0 -0.105579687520261, axis 0.994431640250643 0.105383646114637 0
- added joint right_connect_front: type continuous, parent right_bogie, child right_bogie_front_wheel, origin xyz=0 -0.244262138749221 0.11109638 rpy=0 0 0, axis 1 0 0
