Commit message: urdf ready, gazebo pacakge messed up

File: src/rover_urdf/urdf/chassis_urdf_24.urdf (robot description, URDF)
Before this commit: robot rover_urdf, 11 links, 10 joints
Links:
- link base_link: mass 0.422056388303514 -> None; geometry 
Joints:
- joint left_front_wheel_joint: limit lower=-1.5 upper=1.5 effort=5 velocity=5 -> (none)
