Commit message: IMU still not working, but TF tree is good, and bogie feedback es vale

File: src/rover_urdf/urdf/chassis_urdf_24_gazebo.urdf (robot description, URDF)
Before this commit: robot chassis_24, 11 links, 10 joints
Links:
- added link imu_link, mass 0.01
Joints:
- added joint imu_joint: type fixed, parent chassis_link, child imu_link, origin xyz=0 0 0.1 rpy=0 0 0

Commit message: Camera integrated with the chassis, Video feed integrated into HMI

File: src/rover_urdf/urdf/chassis_urdf_24_gazebo.urdf (robot description, URDF)
Before this commit: robot chassis_24, 12 links, 11 joints
Links:
- added link camera_link, mass 0.01
Joints:
- added joint camera_joint: type fixed, parent chassis_link, child camera_link, origin xyz=0 0 0.5 rpy=0 0 0

Commit message: might be an error

File: src/rover_urdf/urdf/chassis_urdf_24_gazebo.urdf (robot description, URDF)
Before this commit: robot chassis_24, 13 links, 12 joints
Links:
- added link ptz_link, mass 0.01
Joints:
- added joint ptz_joint: type fixed, parent chassis_link, child ptz_link, origin xyz=-0.3 -0.5 0.8 rpy=0 0 0
