Commit message: Required for nav2 atm

File: src/rover_urdf/urdf/chassis_urdf_24_rviz.urdf (robot description, URDF)
Before this commit: robot chassis_24, 11 links, 10 joints
Links:
- added link lidar
Joints:
- added joint lidar_joint: type fixed, parent base_link, child lidar, origin xyz=0 0 0 rpy=0 0 0, axis 0 0 0
