Commit message: renamed rover_urdf to rover_description

File: src/rover_description/urdf/chassis_urdf_24_gazebo.urdf (robot description, URDF)
Before this commit: robot chassis_24, 14 links, 13 joints
Links:
- link back_bogie_link: geometry collision mesh filename=$(find rover_description)/meshes/back_bogie_link.STL; visual mesh filename=$(find rover_description)/meshes/back_bogie_link.STL
- link back_left_wheel_link: geometry collision mesh filename=$(find rover_description)/meshes/back_left_wheel_link.STL; visual mesh filename=$(find rover_description)/meshes/back_left_wheel_link.STL
- link back_right_wheel_link: geometry collision mesh filename=$(find rover_description)/meshes/back_right_wheel_link.STL; visual mesh filename=$(find rover_description)/meshes/back_right_wheel_link.STL
- link chassis_link: geometry collision mesh filename=$(find rover_description)/meshes/chassis_link.STL; visual mesh filename=$(find rover_description)/meshes/chassis_link.STL
- link left_bogie_link: geometry collision mesh filename=$(find rover_description)/meshes/left_bogie_link.STL; visual mesh filename=$(find rover_description)/meshes/left_bogie_link.STL
- link left_front_wheel_link: geometry collision mesh filename=$(find rover_description)/meshes/left_front_wheel_link.STL; visual mesh filename=$(find rover_description)/meshes/left_front_wheel_link.STL
- link left_mid_wheel_link: geometry collision mesh filename=$(find rover_description)/meshes/left_mid_wheel_link.STL; visual mesh filename=$(find rover_description)/meshes/left_mid_wheel_link.STL
- link right_bogie_link: geometry collision mesh filename=$(find rover_description)/meshes/right_bogie_link.STL; visual mesh filename=$(find rover_description)/meshes/right_bogie_link.STL
- link right_front_wheel_link: geometry collision mesh filename=$(find rover_description)/meshes/right_front_wheel_link.STL; visual mesh filename=$(find rover_description)/meshes/right_front_wheel_link.STL
- link right_mid_wheel_link: geometry collision mesh filename=$(find rover_description)/meshes/right_mid_wheel_link.STL; visual mesh filename=$(find rover_description)/meshes/right_mid_wheel_link.STL

File: src/rover_description/urdf/chassis_urdf_24_rviz.urdf (robot description, URDF)
Before this commit: robot chassis_24, 11 links, 10 joints
Links:
- link back_bogie_link: geometry collision mesh filename=package://rover_description/meshes/back_bogie_link.STL; visual mesh filename=package://rover_description/meshes/back_bogie_link.STL
- link back_left_wheel_link: geometry collision mesh filename=package://rover_description/meshes/back_left_wheel_link.STL; visual mesh filename=package://rover_description/meshes/back_left_wheel_link.STL
- link back_right_wheel_link: geometry collision mesh filename=package://rover_description/meshes/back_right_wheel_link.STL; visual mesh filename=package://rover_description/meshes/back_right_wheel_link.STL
- link chassis_link: geometry collision mesh filename=package://rover_description/meshes/chassis_link.STL; visual mesh filename=package://rover_description/meshes/chassis_link.STL
- link left_bogie_link: geometry collision mesh filename=package://rover_description/meshes/left_bogie_link.STL; visual mesh filename=package://rover_description/meshes/left_bogie_link.STL
- link left_front_wheel_link: geometry collision mesh filename=package://rover_description/meshes/left_front_wheel_link.STL; visual mesh filename=package://rover_description/meshes/left_front_wheel_link.STL
- link left_mid_wheel_link: geometry collision mesh filename=package://rover_description/meshes/left_mid_wheel_link.STL; visual mesh filename=package://rover_description/meshes/left_mid_wheel_link.STL
- link right_bogie_link: geometry collision mesh filename=package://rover_description/meshes/right_bogie_link.STL; visual mesh filename=package://rover_description/meshes/right_bogie_link.STL
- link right_front_wheel_link: geometry collision mesh filename=package://rover_description/meshes/right_front_wheel_link.S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; visual mesh filename=package://rover_description/meshes/right_front_wheel_link.S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
- link right_mid_wheel_link: geometry collision mesh filename=package://rover_description/meshes/right_mid_wheel_link.STL; visual mesh filename=package://rover_description/meshes/right_mid_wheel_link.STL
