Commit message: Change to work with imu_filter_madgwick instead of  mahony

File: src/rover_description/urdf/Chassis_jan25.SLDASM.urdf (robot description, URDF)
Before this commit: robot Chassis_jan25.SLDASM, 11 links, 10 joints
Links:
- removed link IMU
- added link imu_link, mass 0.00902500000000001; collision mesh filename=package://Chassis_jan25.SLDASM/meshes/IMU.STL; visual mesh filename=package://Chassis_jan25.SLDASM/meshes/IMU.STL
Joints:
- joint IMU1: child IMU -> imu_link

Commit message: fix urdf temporarily

File: src/rover_description/urdf/Chassis_jan25.SLDASM.urdf (robot description, URDF)
Before this commit: robot Chassis_jan25.SLDASM, 11 links, 10 joints
Links:
- added link lidar
Joints:
- added joint lidar_joint: type fixed, parent base_link, child lidar, origin xyz=0 0 0 rpy=0 0 0

Commit message: Armant/fix local ukf (#100)
* Change to work with imu_filter_madgwick instead of  mahony

* Put all launch stuff in one file

* fix urdf temporarily

File: src/rover_description/urdf/Chassis_jan25.SLDASM.urdf (robot description, URDF)
Before this commit: robot Chassis_jan25.SLDASM, 11 links, 10 joints
Links:
- removed link IMU
- added link imu_link, mass 0.00902500000000001; collision mesh filename=package://Chassis_jan25.SLDASM/meshes/IMU.STL; visual mesh filename=package://Chassis_jan25.SLDASM/meshes/IMU.STL
- added link lidar
Joints:
- added joint lidar_joint: type fixed, parent base_link, child lidar, origin xyz=0 0 0 rpy=0 0 0
- joint IMU1: child IMU -> imu_link
