Commit message: update

File: src/rover_description/urdf/chassis26.urdf (robot description, URDF)
Before this commit: robot Chassis_jan25.SLDASM, 12 links, 11 joints
Links:
- removed link imu_link
- removed link lidar
- added link IMU, mass 0.00902500000000001; collision mesh filename=package://Chassis_jan25.SLDASM/meshes/IMU.STL; visual mesh filename=package://Chassis_jan25.SLDASM/meshes/IMU.STL
Joints:
- removed joint lidar_joint
- joint IMU1: child imu_link -> IMU
