Commit message: Renamed dev_arm package to dev_arm_description

File: src/dev_arm_description/urdf/dev_arm.urdf (robot description, URDF)
Before this commit: robot dev_arm, 9 links, 8 joints
Links:
- link link_0: geometry collision mesh filename=package://dev_arm_description/meshes/link_0.STL; visual mesh filename=package://dev_arm_description/meshes/link_0.STL
- link link_1: geometry collision mesh filename=package://dev_arm_description/meshes/link_1.STL; visual mesh filename=package://dev_arm_description/meshes/link_1.STL
- link link_2: geometry collision mesh filename=package://dev_arm_description/meshes/link_2.STL; visual mesh filename=package://dev_arm_description/meshes/link_2.STL
- link link_3: geometry collision mesh filename=package://dev_arm_description/meshes/link_3.STL; visual mesh filename=package://dev_arm_description/meshes/link_3.STL
- link link_4: geometry collision mesh filename=package://dev_arm_description/meshes/link_4.STL; visual mesh filename=package://dev_arm_description/meshes/link_4.STL
- link link_5: geometry collision mesh filename=package://dev_arm_description/meshes/link_5.STL; visual mesh filename=package://dev_arm_description/meshes/link_5.STL
- link link_6: geometry collision mesh filename=package://dev_arm_description/meshes/link_6.STL; visual mesh filename=package://dev_arm_description/meshes/link_6.STL
- link link_ee: geometry collision mesh filename=package://dev_arm_description/meshes/link_ee.STL; visual mesh filename=package://dev_arm_description/meshes/link_ee.STL

Commit message: dev_arm_description now has a moving ee! No moveit/control integration yet tho

File: src/dev_arm_description/urdf/dev_arm.urdf (robot description, URDF)
Before this commit: robot dev_arm, 9 links, 8 joints
Links:
- removed link link_ee
- added link ee_base_link, mass 0.110400636457142; collision mesh filename=package://dev_arm_description/meshes/ee_base_link.STL; visual mesh filename=package://dev_arm_description/meshes/ee_base_link.STL
- added link finger_left, mass 0.115999619262241; collision mesh filename=package://dev_arm_description/meshes/finger_left.STL; visual mesh filename=package://dev_arm_description/meshes/finger_left.STL
- added link finger_right, mass 0.115999628451242; collision mesh filename=package://dev_arm_description/meshes/finger_right.STL; visual mesh filename=package://dev_arm_description/meshes/finger_right.STL
Joints:
- added joint finger_left_joint: type prismatic, parent ee_base_link, child finger_right, origin xyz=-0.23241 0.37651 0.0074738 rpy=-3.0542 -0.36707 2.5976, axis -0.32112 0.14724 0.93552, limit lower=-1 upper=1 effort=1 velocity=1
- added joint finger_right_joint: type prismatic, parent ee_base_link, child finger_left, origin xyz=-0.25101 0.39517 0.094886 rpy=-0.087358 0.36707 -0.54398, axis 0.32112 0.14724 -0.93552, limit lower=-1 upper=1 effort=1 velocity=1
- joint joint_ee: child link_ee -> ee_base_link; origin xyz=-0.073337 -0.033291 0.14226 rpy=-3.1416 0 1.6469 -> xyz=0.0 0.0145 0.078 rpy=0 -1.5707963 0

Commit message: Got end effector in the right spot, and limits correct Possible prob: the end effector has reduntant stls with axis 6. so theres like 2 axis 6 stls in the same spot

File: src/dev_arm_description/urdf/dev_arm.urdf (robot description, URDF)
Before this commit: robot dev_arm, 11 links, 10 joints
Joints:
- joint finger_left_joint: limit lower=-1 upper=1 effort=1 velocity=1 -> lower=-0.0325 upper=0.061 effort=1 velocity=1
- joint finger_right_joint: limit lower=-1 upper=1 effort=1 velocity=1 -> lower=-0.061 upper=0.0325 effort=1 velocity=1
