Commit message: edited dev_arm_moveit_config_v2 to include gripper

File: src/dev_arm_moveit_config_v2/config/dev_arm.ros2_control.xacro (robot description, xacro)
@@ -50,4 +50,18 @@
                 <state_interface name="velocity"/>
             </joint>
+            <joint name="finger_left_joint">
+                <command_interface name="position"/>
+                <state_interface name="position">
+                  <param name="initial_value">${initial_positions['finger_left_joint']}</param>
+                </state_interface>
+                <state_interface name="velocity"/>
+            </joint>
+            <joint name="finger_right_joint">
+                <command_interface name="position"/>
+                <state_interface name="position">
+                  <param name="initial_value">${initial_positions['finger_right_joint']}</param>
+                </state_interface>
+                <state_interface name="velocity"/>
+            </joint>
         </ros2_control>
     </xacro:macro>
