Commit message: added rover2026 controller

File: src/dev_arm_description_v2/urdf/dev_arm.urdf (robot description, URDF)
Before this commit: robot dev_arm, 10 links, 9 joints
Links:
- link ee_base_link: mass 0.628367460355529 -> 0.110400636457142
- link finger_left: mass 0.59189 -> 0.115999619262241
- link finger_right: mass 0 -> 0.115999628451242
Joints:
- joint a4_rotation: limit lower=-1.57 upper=3.14 effort=10 velocity=1.5 -> lower=-1.57 upper=1.57 effort=10 velocity=1.5
- joint finger_left_joint: axis 0 1 0 -> -0.32112 0.14724 0.93552; child finger_left -> finger_right; limit lower=-0.04 upper=0.04 effort=10 velocity=0.5 -> lower=-0.0325 upper=0.061 effort=1 velocity=1; origin xyz=0 0 0 rpy=0 0 0 -> xyz=-0.23241 0.37651 0.0074738 rpy=-3.0542 -0.36707 2.5976
- joint finger_right_joint: axis 0 1 0 -> 0.32112 0.14724 -0.93552; child finger_right -> finger_left; limit lower=-0.04 upper=0.04 effort=10 velocity=0.5 -> lower=-0.061 upper=0.0325 effort=1 velocity=1; origin xyz=0 0 0 rpy=0 0 0 -> xyz=-0.25101 0.39517 0.094886 rpy=-0.087358 0.36707 -0.54398
- joint joint_ee: axis 1.55075 -0.063574 -0.83224 -> 0.55075 -0.063574 -0.83224; origin xyz=0.1 0.0 0.0 rpy=0 1.571 0 -> xyz=0.0 0.0145 0.078 rpy=0 -1.5707963 0
- joint link1_link2: limit lower=-3.14 upper=3.14 effort=10 velocity=1.5 -> lower=0 upper=3.14 effort=10 velocity=1.5
- joint shoulder_joint: limit lower=-3.14 upper=3.14 effort=10 velocity=1.5 -> lower=-0.22 upper=5.5 effort=10 velocity=1.5; type continuous -> revolute

Commit message: created arm controller for rover2026 and created bus between ros and mujoco

File: src/dev_arm_description_v2/urdf/dev_arm.urdf (robot description, URDF)
Before this commit: robot dev_arm, 10 links, 9 joints
Links:
- link ee_base_link: mass 0.110400636457142 -> 0.628367460355529
- link finger_left: mass 0.115999619262241 -> 0.59189
- link finger_right: mass 0.115999628451242 -> 0
Joints:
- joint finger_left_joint: axis -0.32112 0.14724 0.93552 -> 0 1 0; child finger_right -> finger_left; limit lower=-0.0325 upper=0.061 effort=1 velocity=1 -> lower=0 upper=0 effort=0 velocity=0; origin xyz=-0.23241 0.37651 0.0074738 rpy=-3.0542 -0.36707 2.5976 -> xyz=0 0 0 rpy=0 0 0
- joint finger_right_joint: axis 0.32112 0.14724 -0.93552 -> 0 1 0; child finger_left -> finger_right; limit lower=-0.061 upper=0.0325 effort=1 velocity=1 -> lower=0 upper=0 effort=0 velocity=0; origin xyz=-0.25101 0.39517 0.094886 rpy=-0.087358 0.36707 -0.54398 -> xyz=0 0 0 rpy=0 0 0
- joint joint_ee: axis 0.55075 -0.063574 -0.83224 -> 1.55075 -0.063574 -0.83224; origin xyz=0.0 0.0145 0.078 rpy=0 -1.5707963 0 -> xyz=0.1 0.0 0.0 rpy=0 1.571 0

Commit message: modifying IK for cartesian movement pt1

File: src/dev_arm_description_v2/urdf/dev_arm.urdf (robot description, URDF)
Before this commit: robot dev_arm, 10 links, 9 joints
Joints:
- joint finger_left_joint: limit lower=0 upper=0 effort=0 velocity=0 -> lower=-0.04 upper=0.04 effort=10 velocity=0.5
- joint finger_right_joint: limit lower=0 upper=0 effort=0 velocity=0 -> lower=-0.04 upper=0.04 effort=10 velocity=0.5

File: src/dev_arm_moveit_config_v2/config/dev_arm.urdf.xacro (robot description, xacro)
@@ -2,6 +2,6 @@
 <robot xmlns:xacro="http://www.ros.org/wiki/xacro" name="dev_arm">
     <xacro:arg name="initial_positions_file" default="initial_positions.yaml" />
-    <!-- Import dev_arm urdf file -->
-    <xacro:include filename="$(find dev_arm_moveit_config)/config/dev_arm.urdf.xacro" />
+    <!-- Import dev_arm urdf file (old arm, from dev_arm_description) -->
+    <xacro:include filename="$(find dev_arm_description)/urdf/dev_arm.urdf" />
     <!-- Import control_xacro -->
     <xacro:include filename="dev_arm.ros2_control.xacro" />

Commit message: initial IK commit

File: src/dev_arm_description_v2/urdf/dev_arm.urdf (robot description, URDF)
Before this commit: robot dev_arm, 10 links, 9 joints
Joints:
- joint a4_rotation: limit lower=-1.57 upper=1.57 effort=10 velocity=1.5 -> lower=-1.57 upper=3.14 effort=10 velocity=1.5
- joint link1_link2: limit lower=0 upper=3.14 effort=10 velocity=1.5 -> lower=-3.14 upper=3.14 effort=10 velocity=1.5
- joint shoulder_joint: limit lower=-0.22 upper=5.5 effort=10 velocity=1.5 -> lower=-3.14 upper=3.14 effort=10 velocity=1.5; type revolute -> continuous

Commit message: fixed joy_arm_control from moveit_control

File: src/dev_arm_description_v2/urdf/dev_arm.urdf (robot description, URDF)
Before this commit: robot dev_arm, 10 links, 9 joints
Joints:
- joint a6_rotation: limit lower=0 upper=0 effort=10 velocity=1.5 -> effort=10 velocity=1.5

Commit message: cleaning up

File: src/dev_arm_description_v2/urdf/dev_arm.urdf (robot description, URDF)
Before this commit: robot dev_arm, 10 links, 9 joints
Links:
- added link keyboard, mass 0.5; collision box size=0.102 0.235 0.018; visual mesh filename=package://dev_arm_description_v2/meshes/keyboard_combined.s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
Joints:
- added joint keyboard_joint: type fixed, parent base_link, child keyboard, origin xyz=0.7 0.25 0.009 rpy=0 0 0
